Commit message: Add files via upload

File: scout/scout_description/urdf/VLP-16.urdf.xacro (robot description, xacro)
@@ -17,5 +17,5 @@
     max_angle:=${M_PI}
     gpu:=false">
-    <!-- 雷达支架 -->
+    <!-- 雷达、支架属性 -->
     <xacro:property name="support_length" value="0.30" /> <!-- 支架长度 -->
     <xacro:property name="support_radius" value="0.025" /> <!-- 支架半径 -->
@@ -24,4 +24,9 @@
     <xacro:property name="support_z_size" value="0.255" /> <!-- 支架安装的z坐标:底盘高度 / 2 + 支架高度 / 2  -->
     <xacro:property name="support_m" value="0.02" /> <!-- 支架质量 -->
+    <xacro:property name="laser_length" value="0.0717" /> <!-- laser长度 -->
+    <xacro:property name="laser_radius" value="0.0516" /> <!-- laser半径 -->
+    <xacro:property name="laser_z_size" value="0.255" /> <!-- 支架安装的z坐标:底盘高度 / 2 + 支架高度 / 2  -->
+    <xacro:property name="laser_m" value="0.83" /> <!-- laser质量 -->
+    <!-- 雷达支架 -->
     <link name="support">
         <visual>
@@ -52,24 +57,24 @@
   <!-- 雷达关节以及link -->
     <joint name="${laser_name}_base_mount_joint" type="fixed">
-      <xacro:insert_block name="origin" />
-      <parent link="${out_parent}"/>
-      <child link="${laser_name}_base_link"/>
+        <xacro:insert_block name="origin" />
+        <parent link="${out_parent}"/>
+        <child link="${laser_name}_base_link"/>
     </joint>
     <link name="${laser_name}_base_link">
-      <inertial>
-        <mass value="0.83"/>
-        <origin xyz="0 0 0.03585"/>
-        <inertia ixx="${(0.83 * (3.0*0.0516*0.0516 + 0.0717*0.0717)) / 12.0}" ixy="0" ixz="0"
-          iyy="${(0.83 * (3.0*0.0516*0.0516 + 0.0717*0.0717)) / 12.0}" iyz="0"
-          izz="${0.5 * 0.83 * (0.0516*0.0516)}"/>
-      </inertial>
+        <inertial>
+            <mass value="0.83"/>
+            <origin xyz="0 0 0.03585"/>
+            <inertia ixx="${(0.83 * (3.0*0.0516*0.0516 + 0.0717*0.0717)) / 12.0}" ixy="0" ixz="0"
+                    iyy="${(0.83 * (3.0*0.0516*0.0516 + 0.0717*0.0717)) / 12.0}" iyz="0"
+                    izz="${0.5 * 0.83 * (0.0516*0.0516)}"/>
+        </inertial>
       <visual>
         <geometry>
-          <mesh filename="package://scout_description/meshes/VLP16_base_1.dae" />
+            <mesh filename="package://scout_description/meshes/VLP16_base_1.dae" />
         </geometry>
       </visual>
       <visual>
         <geometry>
-          <mesh filename="package://scout_description/meshes/VLP16_base_2.dae" />
+            <mesh filename="package://scout_description/meshes/VLP16_base_2.dae" />
         </geometry>
       </visual>
@@ -77,108 +82,108 @@
         <origin rpy="0 0 0" xyz="0 0 0.03585"/>
         <geometry>
-          <cylinder radius="0.0516" length="0.0717"/>
+            <cylinder radius="0.0516" length="0.0717"/>
         </geometry>
       </collision>
     </link>
     <joint name="${laser_name}_base_scan_joint" type="fixed" >
-      <origin xyz="0 0 0.0377" rpy="0 0 0" />
-      <parent link="${laser_name}_base_link" />
-      <child link="${laser_name}"/>
+        <origin xyz="0 0 0.0377" rpy="0 0 0" />
+        <parent link="${laser_name}_base_link" />
+        <child link="${laser_name}"/>
     </joint>
     <link name="${laser_name}">
-      <inertial>
-        <mass value="0.01"/>
-        <origin xyz="0 0 0"/>
-        <inertia ixx="1e-7" ixy="0" ixz="0" iyy="1e-7" iyz="0" izz="1e-7"/>
-      </inertial>
-      <visual>
-        <origin xyz="0 0 -0.0377" />
-        <geometry>
-          <mesh filename="package://scout_description/meshes/VLP16_scan.dae" />
-        </geometry>
-      </visual>
+        <inertial>
+            <mass value="0.01"/>
+            <origin xyz="0 0 0"/>
+            <inertia ixx="1e-7" ixy="0" ixz="0" iyy="1e-7" iyz="0" izz="1e-7"/>
+        </inertial>
+        <visual>
+            <origin xyz="0 0 -0.0377" />
+            <geometry>
+                <mesh filename="package://scout_description/meshes/VLP16_scan.dae" />
+            </geometry>
+        </visual>
     </link>
     <!-- Gazebo requires the velodyne_gazebo_plugins package -->
     <gazebo reference="${laser_name}">
-      <xacro:if value="${gpu}">
-        <sensor type="gpu_ray" name="${laser_name}-VLP16">
-          <pose>0 0 0 0 0 0</pose>
-          <visualize>false</visualize>
-          <update_rate>${hz}</update_rate>
-          <ray>
-            <scan>
-              <horizontal>
-                <samples>${samples}</samples>
-                <resolution>1</resolution>
-                <min_angle>${min_angle}</min_angle>
-                <max_angle>${max_angle}</max_angle>
-              </horizontal>
-              <vertical>
-                <samples>${lasers}</samples>
-                <resolution>1</resolution>
-                <min_angle>-${15.0*M_PI/180.0}</min_angle>
-                <max_angle> ${15.0*M_PI/180.0}</max_angle>
-              </vertical>
-            </scan>
-            <range>
-              <min>${collision_range}</min>
-              <max>${max_range+1}</max>
-              <resolution>0.001</resolution>
-            </range>
-            <noise>
-              <type>gaussian</type>
-              <mean>0.0</mean>
-              <stddev>0.0</stddev>
-            </noise>
-          </ray>
-          <plugin name="gazebo_ros_laser_controller" filename="libgazebo_ros_velodyne_gpu_laser.so">
-            <topicName>${topic}</topicName>
-            <frameName>${laser_name}</frameName>
-            <organize_cloud>${organize_cloud}</organize_cloud>
-            <min_range>${min_range}</min_range>
-            <max_range>${max_range}</max_range>
-            <gaussianNoise>${noise}</gaussianNoise>
-          </plugin>
-        </sensor>
-      </xacro:if>
+        <xacro:if value="${gpu}">
+            <sensor type="gpu_ray" name="${laser_name}-VLP16">
+            <pose>0 0 0 0 0 0</pose>
+            <visualize>false</visualize>
+            <update_rate>${hz}</update_rate>
+                <ray>
+                    <scan>
+                    <horizontal>
+                        <samples>${samples}</samples>
+                        <resolution>1</resolution>
+                        <min_angle>${min_angle}</min_angle>
+                        <max_angle>${max_angle}</max_angle>
+                    </horizontal>
+                    <vertical>
+                        <samples>${lasers}</samples>
+                        <resolution>1</resolution>
+                        <min_angle>-${15.0*M_PI/180.0}</min_angle>
+                        <max_angle> ${15.0*M_PI/180.0}</max_angle>
+                    </vertical>
+                    </scan>
+                    <range>
+                    <min>${collision_range}</min>
+                    <max>${max_range+1}</max>
+                    <resolution>0.001</resolution>
+                    </range>
+                    <noise>
+                    <type>gaussian</type>
+                    <mean>0.0</mean>
+                    <stddev>0.0</stddev>
+                    </noise>
+                </ray>
+                <plugin name="gazebo_ros_laser_controller" filename="libgazebo_ros_velodyne_gpu_laser.so">
+                    <topicName>${topic}</topicName>
+                    <frameName>${laser_name}</frameName>
+                    <organize_cloud>${organize_cloud}</organize_cloud>
+                    <min_range>${min_range}</min_range>
+                    <max_range>${max_range}</max_range>
+                    <gaussianNoise>${noise}</gaussianNoise>
+                </plugin>
+            </sensor>
+        </xacro:if>
       <xacro:unless value="${gpu}">
         <sensor type="ray" name="${laser_name}-VLP16">
-          <pose>0 0 0 0 0 0</pose>
-          <visualize>false</visualize>
-          <update_rate>${hz}</update_rate>
-          <ray>
-            <scan>
-              <horizontal>
-                <samples>${samples}</samples>
-                <resolution>1</resolution>
-                <min_angle>${min_angle}</min_angle>
-                <max_angle>${max_angle}</max_angle>
-              </horizontal>
-              <vertical>
-                <samples>${lasers}</samples>
-                <resolution>1</resolution>
-                <min_angle>-${15.0*M_PI/180.0}</min_angle>
-                <max_angle> ${15.0*M_PI/180.0}</max_angle>
-              </vertical>
-            </scan>
-            <range>
-              <min>${collision_range}</min>
-              <max>${max_range+1}</max>
-              <resolution>0.001</resolution>
-            </range>
-            <noise>
-              <type>gaussian</type>
-              <mean>0.0</mean>
-              <stddev>0.0</stddev>
-            </noise>
-          </ray>
-          <plugin name="gazebo_ros_laser_controller" filename="libgazebo_ros_velodyne_laser.so">
-            <topicName>${topic}</topicName>
-            <frameName>${laser_name}</frameName>
-            <organize_cloud>${organize_cloud}</organize_cloud>
-            <min_range>${min_range}</min_range>
-            <max_range>${max_range}</max_range>
-            <gaussianNoise>${noise}</gaussianNoise>
-          </plugin>
+            <pose>0 0 0 0 0 0</pose>
+            <visualize>false</visualize>
+            <update_rate>${hz}</update_rate>
+            <ray>
+                <scan>
+                    <horizontal>
+                        <samples>${samples}</samples>
+                        <resolution>1</resolution>
+                        <min_angle>${min_angle}</min_angle>
+                        <max_angle>${max_angle}</max_angle>
+                    </horizontal>
+                    <vertical>
+                        <samples>${lasers}</samples>
+                        <resolution>1</resolution>
+                        <min_angle>-${15.0*M_PI/180.0}</min_angle>
+                        <max_angle> ${15.0*M_PI/180.0}</max_angle>
+                    </vertical>
+                </scan>
+                <range>
+                    <min>${collision_range}</min>
+                    <max>${max_range+1}</max>
+                    <resolution>0.001</resolution>
+                </range>
+                <noise>
+                    <type>gaussian</type>
+                    <mean>0.0</mean>
+                    <stddev>0.0</stddev>
+                </noise>
+            </ray>
+            <plugin name="gazebo_ros_laser_controller" filename="libgazebo_ros_velodyne_laser.so">
+                <topicName>${topic}</topicName>
+                <frameName>${laser_name}</frameName>
+                <organize_cloud>${organize_cloud}</organize_cloud>
+                <min_range>${min_range}</min_range>
+                <max_range>${max_range}</max_range>
+                <gaussianNoise>${noise}</gaussianNoise>
+            </plugin>
         </sensor>
       </xacro:unless>

File: scout/scout_description/urdf/camera.xacro (robot description, xacro)
@@ -33,5 +33,43 @@
     </joint>
     <gazebo reference="camera">
-        <material>Gazebo/Blue</material>
+        <material>Gazebo/Black</material>
+    </gazebo>
+	<!-- gazebo相机插件配置 -->
+    <gazebo reference="camera">
+        <sensor type="camera" name="camera_node">
+            <update_rate>30.0</update_rate> <!-- 更新频率 -->
+            <camera name="head"><!-- 摄像头基本信息设置 -->
+                <horizontal_fov>1.3962634</horizontal_fov>
+                <image>
+                    <width>1280</width>
+                    <height>720</height>
+                    <format>R8G8B8</format>
+                </image>
+                <clip>
+                    <near>0.02</near>
+                    <far>300</far>
+                </clip>
+                <noise>
+                    <type>gaussian</type>
+                    <mean>0.0</mean>
+                    <stddev>0.007</stddev>
+                </noise>
+            </camera>
+            <!-- 核心插件 -->
+            <plugin name="gazebo_camera" filename="libgazebo_ros_camera.so">
+                <alwaysOn>true</alwaysOn>
+                <updateRate>0.0</updateRate>
+                <cameraName>/camera</cameraName>
+                <imageTopicName>image_raw</imageTopicName>
+                <cameraInfoTopicName>camera_info</cameraInfoTopicName>
+                <frameName>camera</frameName>
+                <hackBaseline>0.07</hackBaseline>
+                <distortionK1>0.0</distortionK1>
+                <distortionK2>0.0</distortionK2>
+                <distortionK3>0.0</distortionK3>
+                <distortionT1>0.0</distortionT1>
+                <distortionT2>0.0</distortionT2>
+            </plugin>
+        </sensor>
     </gazebo>
 </robot>

File: scout/scout_description/urdf/combination.xacro (robot description, xacro)
@@ -6,11 +6,10 @@
   <xacro:property name="organize_cloud" value="$(arg organize_cloud)" />
 	<!-- include -->
-	<xacro:include filename="$(find scout_description)/urdf/inertial.xacro" /><!--惯性矩阵计算模块-->+
+	<xacro:include filename="$(find scout_description)/urdf/inertial.xacro" /><!--惯性矩阵计算模块-->
 	<xacro:include filename="$(find scout_description)/urdf/scout_v2.xacro" /><!--底盘模块-->
   <!--<xacro:include filename="$(find scout_description)/urdf/laser.xacro" />单线激光雷达-->
-  <!--<xacro:include filename="$(find scout_description)/urdf/sensor_laser.xacro" />单线激光雷达-->
 	<xacro:include filename="$(find scout_description)/urdf/camera.xacro" /><!--相机模块-->
-  <xacro:include filename="$(find scout_description)/urdf/sensor_camera.xacro" /><!--相机感知模块-->
   <xacro:include filename="$(find scout_description)/urdf/VLP-16.urdf.xacro"/><!--16线激光雷达模块-->
+  <xacro:include filename="$(find scout_description)/urdf/IMU.xacro" /><!--imu模块-->
   <xacro:VLP-16 out_parent="base_link" laser_name="velodyne" topic="/velodyne_points" organize_cloud="${organize_cloud}" hz="10" samples="440" gpu="${gpu}">
     <origin xyz="0 0 0.4" rpy="0 0 0" />

File: scout/scout_description/urdf/inertial.xacro (robot description, xacro)
@@ -1,2 +1,3 @@
+<?xml version="1.0"?>
 <robot name="base" xmlns:xacro="http://wiki.ros.org/xacro">
     <!-- Macro for inertia matrix -->

File: scout/scout_description/urdf/laser.xacro (robot description, xacro)
@@ -2,5 +2,11 @@
 <!--小车底盘添加雷达-->
 <robot name="my_laser" xmlns:xacro="http://wiki.ros.org/xacro">
-    <!-- 雷达支架 -->
+    <!-- 雷达及支架属性 -->
+    <xacro:property name="laser_length" value="0.05" /> <!-- 雷达长度 -->
+    <xacro:property name="laser_radius" value="0.07" /> <!-- 雷达半径 -->
+    <xacro:property name="laser_x" value="0.0" /> <!-- 雷达安装的x坐标 -->
+    <xacro:property name="laser_y" value="0.0" /> <!-- 雷达安装的y坐标 -->
+    <xacro:property name="laser_z" value="0.175" /> <!-- 雷达安装的z坐标:支架高度 / 2 + 雷达高度 / 2  -->
+    <xacro:property name="laser_m" value="0.1" /> <!-- 雷达质量 -->
     <xacro:property name="support_length" value="0.30" /> <!-- 支架长度 -->
     <xacro:property name="support_radius" value="0.025" /> <!-- 支架半径 -->
@@ -9,4 +15,5 @@
     <xacro:property name="support_z_size" value="0.255" /> <!-- 支架安装的z坐标:底盘高度 / 2 + 支架高度 / 2  -->
     <xacro:property name="support_m" value="0.02" /> <!-- 支架质量 -->
+    <!-- 雷达支架 -->
     <link name="support">
         <visual>
@@ -32,15 +39,5 @@
         <origin xyz="${support_x_size} ${support_y_size} ${support_z_size}" />
     </joint>
-    <gazebo reference="support">
-        <material>Gazebo/White</material>
-    </gazebo>
-    <!-- 雷达属性 -->
-    <xacro:property name="laser_length" value="0.05" /> <!-- 雷达长度 -->
-    <xacro:property name="laser_radius" value="0.07" /> <!-- 雷达半径 -->
-    <xacro:property name="laser_x" value="0.0" /> <!-- 雷达安装的x坐标 -->
-    <xacro:property name="laser_y" value="0.0" /> <!-- 雷达安装的y坐标 -->
-    <xacro:property name="laser_z" value="0.175" /> <!-- 雷达安装的z坐标:支架高度 / 2 + 雷达高度 / 2  -->
-    <xacro:property name="laser_m" value="0.1" /> <!-- 雷达质量 -->
-    <!-- 雷达关节以及link -->
+    <!-- 雷达 -->
     <link name="laser">
         <visual>
@@ -64,6 +61,35 @@
         <origin xyz="${laser_x} ${laser_y} ${laser_z}" />
     </joint>
+	<!-- gazebo雷达插件配置 -->
     <gazebo reference="laser">
-        <material>Gazebo/Black</material>
+        <sensor type="ray" name="rplidar">
+        <pose>0 0 0 0 0 0</pose>
+        <visualize>true</visualize>
+        <update_rate>5.5</update_rate>
+            <ray>
+                <scan>
+                <horizontal>
+                    <samples>360</samples>
+                    <resolution>1</resolution>
+                    <min_angle>-3</min_angle>
+                    <max_angle>3</max_angle>
+                </horizontal>
+                </scan>
+                <range>
+                <min>0.10</min>
+                <max>30.0</max>
+                <resolution>0.01</resolution>
+                </range>
+                <noise>
+                <type>gaussian</type>
+                <mean>0.0</mean>
+                <stddev>0.01</stddev>
+                </noise>
+            </ray>
+            <plugin name="gazebo_rplidar" filename="libgazebo_ros_laser.so">
+                <topicName>/scan</topicName>
+                <frameName>laser</frameName>
+            </plugin>
+        </sensor>
     </gazebo>
 </robot>

Commit message: Add files via upload

File: scout/scout_description/urdf/VLP-16.urdf.xacro (robot description, xacro)
@@ -68,4 +68,7 @@
                     iyy="${(0.83 * (3.0*0.0516*0.0516 + 0.0717*0.0717)) / 12.0}" iyz="0"
                     izz="${0.5 * 0.83 * (0.0516*0.0516)}"/>
+            <inertia ixx="${laser_m*(3*laser_radius*laser_radius+laser_length*laser_length)/12}" ixy = "0" ixz = "0"
+                    iyy="${laser_m*(3*laser_radius*laser_radius+laser_length*laser_length)/12}" iyz = "0"
+                    izz="${laser_m*laser_radius*laser_radius/2}" />
         </inertial>
       <visual>

File: scout/scout_description/urdf/scout_v2.xacro (robot description, xacro)
@@ -15,4 +15,5 @@
     <xacro:property name="wheel_length" value="1.1653e-01" />
     <xacro:property name="wheel_radius" value="1.6459e-01" />
+    <xacro:property name="mass" value="5000" />
      <!-- include -->
     <xacro:include filename="$(find scout_description)/urdf/scout_wheel_type1.xacro" />
@@ -46,10 +47,12 @@
     <link name="inertial_link">
         <inertial>
-            <mass value="50" />
+            <mass value="${mass}" />
             <!-- <mass value="50" /> -->
             <!-- <origin xyz="-0.00065 -0.085 0.062" />
             <inertia ixx="0.6022" ixy="-0.02364" ixz="-0.1197" iyy="1.7386" iyz="-0.001544" izz="2.0296" /> -->
             <origin xyz="0.0 0.0 0.0" />
-            <inertia ixx="2.288641" ixy="0" ixz="0" iyy="5.103976" iyz="0" izz="3.431465" />
+            <inertia ixx="${mass*(base_z_size*base_z_size + base_x_size*base_x_size)/12}" ixy = "0" ixz = "0"
+                   iyy="${mass*(base_y_size*base_y_size + base_x_size*base_x_size)/12}" iyz= "0"
+                   izz="${mass*(base_y_size*base_y_size + base_z_size*base_z_size)/12}" />
         </inertial>
     </link>
